File: pcb/adelheid.sch (KiCad schematic (older format))
At the start: 40 parts, among them J1 USB_B_Mini, J12 VCC, J13 D+, J14 D-, J15 GND, J2 MISO, J3 VCC, J4 SCK, J5 MOSI, J6 RES, J7 GND, J8 PF4, J9 PF5, Q1 2N7002, U1 USBLC6-2SC6, U2 ATmega32U4-AU, Y1 Crystal_GND24

Commit message: Converted Adelheid mini USB to Aristutea USB-C
Parts:
- removed J1: USB_B_Mini, Keebio-Parts:USB-Mini-B_2leg, symbol Connector:USB_B_Micro
- removed J14: D-, Pin_Headers:Pin_Header_Straight_1x01_Pitch2.54mm, symbol Connector_Generic:Conn_01x01
- removed J15: GND, Pin_Headers:Pin_Header_Straight_1x01_Pitch2.54mm, symbol Connector_Generic:Conn_01x01
- added J1: USB_C_Receptacle_HRO_TYPE-C-31-M-12, arisutea:USB_C_Receptacle_HRO_TYPE-C-31-M-12-HandSoldering, symbol USB_Type-C:USB_C_Receptacle_HRO_TYPE-C-31-M-12
- added J10: D-, Connector_PinHeader_2.54mm:PinHeader_1x01_P2.54mm_Vertical, symbol Connector_Generic:Conn_01x01
- added J11: D+, Connector_PinHeader_2.54mm:PinHeader_1x01_P2.54mm_Vertical, symbol Connector_Generic:Conn_01x01
- added R6, R7: 22, Resistor_SMD:R_0805_2012Metric_Pad1.20x1.40mm_HandSolder, symbol Device:R
- J12: footprint Pin_Headers:Pin_Header_Straight_1x01_Pitch2.54mm -> Connector_PinHeader_2.54mm:PinHeader_1x01_P2.54mm_Vertical
- J13: value D+ -> GND; footprint Pin_Headers:Pin_Header_Straight_1x01_Pitch2.54mm -> Connector_PinHeader_2.54mm:PinHeader_1x01_P2.54mm_Vertical
- R1, R2: value 22 -> 5K1; footprint Resistor_SMD:R_0805_2012Metric_Pad1.15x1.40mm_HandSolder -> arisutea:R_0805_2012Metric_Pad1.20x1.40mm_HandSolder
- U1: footprint TO_SOT_Packages_SMD:SOT-23-6_Handsoldering -> Package_TO_SOT_SMD:SOT-23-6_Handsoldering
Connections:
- wire segments 143 -> 135
- no-connect marks 4 -> 3
