File: pcb/adelheid.kicad_pcb (KiCad board)
At the start: 2 copper layers, 339.1 x 143.2 mm, 323 parts, among them J1 USB_B_Mini, J12 VCC, J13 D+, J14 D-, J15 GND, J2 MISO, J3 VCC, J4 SCK, J5 MOSI, J6 RES, J7 GND, J8 PF4, J9 PF5, Q1 2N7002, U1 USBLC6-2SC6, U2 ATmega32U4-AU, Y1 Crystal_GND24

Commit message: WIP: CLeaning up old tracks and starting to layout new components.
Parts:
- removed  G2: LOGO, adelheid:adelheid-logo
- removed G1: LOGO, adelheid:adelheid-logo
- removed J12: VCC, Pin_Headers:Pin_Header_Straight_1x01_Pitch2.54mm
- removed J13: D+, Pin_Headers:Pin_Header_Straight_1x01_Pitch2.54mm
- removed J14: D-, Pin_Headers:Pin_Header_Straight_1x01_Pitch2.54mm
- removed J15, J7: GND, Pin_Headers:Pin_Header_Straight_1x01_Pitch2.54mm
- removed J4: SCK, Pin_Headers:Pin_Header_Straight_1x01_Pitch2.54mm
- removed J5: MOSI, Pin_Headers:Pin_Header_Straight_1x01_Pitch2.54mm
- removed J6: RES, Pin_Headers:Pin_Header_Straight_1x01_Pitch2.54mm
- removed J8: PF4, Pin_Headers:Pin_Header_Straight_1x01_Pitch2.54mm
- removed J9: PF5, Pin_Headers:Pin_Header_Straight_1x01_Pitch2.54mm
- removed LS1, LS10, LS11, LS12, LS13, LS14, LS15, LS16, LS17, LS2, LS3, LS4, LS5, LS6, LS7, LS8, LS9: LED, LED_SMD:LED_0805_2012Metric_Pad1.15x1.40mm_HandSolder
- removed RS1, RS10, RS11, RS12, RS13, RS14, RS15, RS16, RS17, RS2, RS3, RS4, RS5, RS6, RS7, RS8, RS9: R, Resistor_SMD:R_0805_2012Metric_Pad1.15x1.40mm_HandSolder
- added D83: WS2812B, LED_SMD:LED_WS2812B_PLCC4_5.0x5.0mm_P3.2mm, B.Cu at (49.3, 16.5)
- added D84: WS2812B, LED_SMD:LED_WS2812B_PLCC4_5.0x5.0mm_P3.2mm, B.Cu at (16.5, 54.9)
- added D85: WS2812B, LED_SMD:LED_WS2812B_PLCC4_5.0x5.0mm_P3.2mm, B.Cu at (14.7, 88.9)
- added D86: WS2812B, LED_SMD:LED_WS2812B_PLCC4_5.0x5.0mm_P3.2mm, B.Cu at (16.5, 121.7)
- added D87: WS2812B, LED_SMD:LED_WS2812B_PLCC4_5.0x5.0mm_P3.2mm, B.Cu at (120.9, 17.5)
- added D88: WS2812B, LED_SMD:LED_WS2812B_PLCC4_5.0x5.0mm_P3.2mm, B.Cu at (68.1, 162.6)
- added D89: WS2812B, LED_SMD:LED_WS2812B_PLCC4_5.0x5.0mm_P3.2mm, B.Cu at (282.4, 18.0)
- added D90: WS2812B, LED_SMD:LED_WS2812B_PLCC4_5.0x5.0mm_P3.2mm, B.Cu at (128.4, 168.8)
- added D91: WS2812B, LED_SMD:LED_WS2812B_PLCC4_5.0x5.0mm_P3.2mm, B.Cu at (177.5, 176.8)
- added D92: WS2812B, LED_SMD:LED_WS2812B_PLCC4_5.0x5.0mm_P3.2mm, B.Cu at (343.7, 17.3)
- added D93: WS2812B, LED_SMD:LED_WS2812B_PLCC4_5.0x5.0mm_P3.2mm, B.Cu at (261.9, 165.4)
- added D94: WS2812B, LED_SMD:LED_WS2812B_PLCC4_5.0x5.0mm_P3.2mm, B.Cu at (372.6, 58.4)
- added D95: WS2812B, LED_SMD:LED_WS2812B_PLCC4_5.0x5.0mm_P3.2mm, B.Cu at (372.1, 101.1)
- added D96: WS2812B, LED_SMD:LED_WS2812B_PLCC4_5.0x5.0mm_P3.2mm, B.Cu at (373.9, 149.4)
- added D97: WS2812B, LED_SMD:LED_WS2812B_PLCC4_5.0x5.0mm_P3.2mm, B.Cu at (318.6, 163.8)
- added R6: 5k1, Resistor_SMD:R_0805_2012Metric_Pad1.20x1.40mm_HandSolder, B.Cu at (182.9, 0.51)
- added R7: 5k1, Resistor_SMD:R_0805_2012Metric_Pad1.20x1.40mm_HandSolder, B.Cu at (190.2, -0.89)
- J1: value USB_B_Mini -> USB_C_Receptacle_HRO_TYPE-C-31-M-12; footprint Keebio-Parts:USB-Mini-B_2leg -> adelheid:USB_C_Receptacle_HRO_TYPE-C-31-M-12-HandSoldering
- J2: value MISO -> Conn_01x06; footprint Pin_Headers:Pin_Header_Straight_1x01_Pitch2.54mm -> Connector_PinHeader_2.54mm:PinHeader_1x06_P2.54mm_Vertical
- J3: value VCC -> Conn_01x06; footprint Pin_Headers:Pin_Header_Straight_1x01_Pitch2.54mm -> Connector_PinHeader_2.54mm:PinHeader_1x06_P2.54mm_Vertical
- moved J2 73.9 mm to (146.8, 26.7), turned to 90 degrees
- moved J1 7.75 mm to (175.2, 22.9)
- moved J3 4.07 mm to (222.2, 26.7), turned to 90 degrees
Connections:
- J2 pad 1: /MISO -> VCC
- J3 pad 1: VCC -> MISO
- MX40 pad 1: /SCK -> SCLK
- MX41 pad 1: /SCK -> SCLK
- MX42 pad 1: /SCK -> SCLK
- MX43 pad 1: /SCK -> SCLK
- MX44 pad 1: /SCK -> SCLK
- MX45 pad 1: /SCK -> SCLK
- MX77 pad 1: /MISO -> MISO
- MX78 pad 1: /MISO -> MISO
- MX79 pad 1: /MISO -> MISO
- MX80 pad 1: /MISO -> MISO
- MX81 pad 1: /MISO -> MISO
- MX82 pad 1: /MISO -> MISO
- R1 pad 2: Net-(J1-Pad3) -> USB+
- R2 pad 2: Net-(J1-Pad2) -> USB-
- R3 pad 2: /~RES~ -> RESET
- SWR1 pad 2: /~RES~ -> RESET
- U1 pad 1: Net-(U1-Pad1) -> Net-(J1-PadA7)
- U1 pad 3: Net-(U1-Pad3) -> Net-(J1-PadA6)
- U1 pad 4: Net-(J1-Pad2) -> USB+
- U1 pad 6: Net-(J1-Pad3) -> USB-
- U2 pad 10: /MOSI -> MOSI
- U2 pad 11: /MISO -> MISO
- U2 pad 13: /~RES~ -> RESET
- U2 pad 38: /PF5 -> PF5
- U2 pad 39: /PF4 -> PF4
- U2 pad 42: Net-(U2-Pad42) -> (no net)
- U2 pad 9: /SCK -> SCLK
Routing:
- net /MISO: track 331.7 -> 0.00 mm, vias 1 -> 0
- net VCC: track 2646.7 -> 2324.3 mm, vias 15 -> 10
- net /SCK: track 197.3 -> 0.00 mm, vias 2 -> 0
- net /ledGND: track 2409.6 -> 2221.1 mm
- net SCLK: track 0.00 -> 177.7 mm, vias 0 -> 1
- net MISO: track 0.00 -> 161.9 mm
- net Net-(J1-Pad3): track 47.7 -> 0.00 mm, vias 2 -> 0
- net Net-(J1-Pad2): track 40.8 -> 0.00 mm, vias 1 -> 0
- net /PF5: track 40.2 -> 0.00 mm, vias 1 -> 0
- net /MOSI: track 39.7 -> 0.00 mm, vias 1 -> 0
- net /PF4: track 38.1 -> 0.00 mm, vias 1 -> 0
- net /~RES~: track 37.0 -> 0.00 mm, vias 2 -> 0
- net RESET: track 0.00 -> 28.3 mm, vias 0 -> 2
- net GND: track 61.7 -> 41.6 mm, vias 21 -> 4
- net Net-(LS4-Pad1): track 3.30 -> 0.00 mm
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
Commit message: Replaced WS21812B with mini version and connected all track. (post clean up commit)
Parts:
- removed MX29: MX-LED, ai03-MX_only:MXOnly-1U
- added D98: WS2812B_Mini, LED_SMD:LED_SK6812MINI_PLCC4_3.5x3.5mm_P1.75mm, B.Cu at (247.7, 26.9)
- D83, D84, D85, D86, D87, D88, D89, D90, D91, D92, D93, D94, D95, D96, D97: value WS2812B -> WS2812B_Mini; footprint LED_SMD:LED_WS2812B_PLCC4_5.0x5.0mm_P3.2mm -> LED_SMD:LED_SK6812MINI_PLCC4_3.5x3.5mm_P1.75mm
- moved D89 216.9 mm to (111.8, 151.9), turned to 168 degrees
- moved D87 143.3 mm to (28.4, 127.0), turned to 90 degrees
- moved D92 139.1 mm to (304.3, 150.7), turned to 180 degrees
- moved D97 138.6 mm to (298.2, 26.7)
- moved D96 124.3 mm to (351.8, 27.1)
- moved D93 106.5 mm to (361.2, 127.0), turned to 270 degrees
- moved D91 70.0 mm to (243.0, 151.9), turned to 192 degrees
- moved D83 66.1 mm to (114.5, 27.3)
- moved D95 61.1 mm to (361.4, 40.9), turned to 270 degrees
- moved D84 58.3 mm to (67.8, 27.2), turned to 0 degrees
- moved D90 47.9 mm to (176.1, 164.5), turned to 180 degrees
- moved D85 40.7 mm to (28.4, 50.5), turned to 90 degrees
- moved D86 37.8 mm to (28.4, 85.9), turned to 90 degrees
- moved R7 37.7 mm to (168.9, 30.2), turned to 90 degrees
- moved D94 29.5 mm to (361.8, 85.9), turned to 270 degrees
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Connections:
- D83 pad 4: Net-(D83-Pad4) -> PF5
- D87 pad 2: Net-(D83-Pad4) -> Net-(D87-Pad2)
- D87 pad 4: Net-(D87-Pad4) -> Net-(D86-Pad2)
- D88 pad 4: Net-(D86-Pad2) -> Net-(D87-Pad2)
- D89 pad 2: Net-(D87-Pad4) -> Net-(D89-Pad2)
- D89 pad 4: PF5 -> Net-(D88-Pad2)
- D90 pad 4: Net-(D88-Pad2) -> Net-(D89-Pad2)
- D92 pad 2: PF5 -> Net-(D92-Pad2)
- D92 pad 4: Net-(D92-Pad4) -> Net-(D91-Pad2)
- D93 pad 4: Net-(D91-Pad2) -> Net-(D92-Pad2)
- D94 pad 2: Net-(D92-Pad4) -> Net-(D94-Pad2)
- D94 pad 4: Net-(D94-Pad4) -> Net-(D93-Pad2)
- D95 pad 2: Net-(D94-Pad4) -> Net-(D95-Pad2)
- D95 pad 4: Net-(D95-Pad4) -> Net-(D94-Pad2)
- D96 pad 2: Net-(D95-Pad4) -> Net-(D96-Pad2)
- D96 pad 4: Net-(D96-Pad4) -> Net-(D95-Pad2)
- D97 pad 2: Net-(D96-Pad4) -> Net-(D97-Pad2)
- D97 pad 4: Net-(D93-Pad2) -> Net-(D96-Pad2)
- J1 pad A4: Net-(J1-PadA4) -> VCC
- J1 pad A9: Net-(J1-PadA4) -> VCC
Routing:
- net VCC: track 2324.3 -> 2726.6 mm, vias 10 -> 16
- net MISO: track 161.9 -> 330.9 mm, vias 0 -> 2
- net GND: track 41.6 -> 134.2 mm, vias 4 -> 3
- net Net-(D92-Pad2): track 0.00 -> 77.5 mm
- net Net-(D89-Pad2): track 0.00 -> 66.5 mm, vias 0 -> 2
- net Net-(D90-Pad2): track 0.00 -> 66.1 mm
- net PF5: track 0.00 -> 62.2 mm, vias 0 -> 2
- net Net-(D91-Pad2): track 0.00 -> 59.6 mm
- net Net-(D88-Pad2): track 0.00 -> 57.9 mm, vias 0 -> 2
- net /ledGND: track 2221.1 -> 2163.9 mm, vias 19 -> 12
- net Net-(D84-Pad2): track 0.00 -> 51.9 mm
- net Net-(D96-Pad2): track 0.00 -> 51.2 mm
- net Net-(D97-Pad2): track 0.00 -> 47.9 mm
- net Net-(D83-Pad2): track 0.00 -> 43.9 mm
- net Net-(D94-Pad2): track 0.00 -> 42.4 mm
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
Commit message: Fixed key that had accidentally been deleted! cleaned up any DRC markers.
Parts:
- added MX29: MX-LED, ai03-MX_only:MXOnly-1U, F.Cu at (143.1, 49.5)
- moved R7 2.29 mm to (168.9, 28.0), turned to 270 degrees
- moved R5 0.72 mm to (155.7, 35.6)
Routing:
- net /ledGND: track 2163.9 -> 2146.8 mm, vias 12 -> 11
- net Net-(D84-Pad2): track 51.9 -> 46.1 mm, vias 0 -> 2
- net /col2: track 219.6 -> 216.3 mm
- net VCC: track 2726.6 -> 2729.8 mm, vias 16 -> 18
- net GND: track 134.2 -> 132.8 mm, vias 3 -> 4
- net MISO: track 330.9 -> 329.5 mm, vias 2 -> 3
- net Net-(R5-Pad1): track 35.1 -> 34.3 mm
- net Net-(Q1-Pad1): track 3.65 -> 4.37 mm
- net Net-(D97-Pad2): track 47.9 -> 48.4 mm
